File: hardware/s105/MPSNG5.kicad_sch (KiCad schematic)
At the start: 9 parts, among them U4 case only

Commit message: +knock
Parts:
- R158: value 47k -> 4.7k
- R204: value 1K -> 100
Changed lines of the file:
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@@
     (in_bom yes) (on_board yes)
     (property "Reference" "R158" (id 0) (at 154.305 93.98 90))
-    (property "Value" "47k" (id 1) (at 154.305 91.44 90))
+    (property "Value" "4.7k" (id 1) (at 154.305 91.44 90))
     (property "Footprint" "Resistor_SMD:R_0603_1608Metric" (id 2) (at 154.305 89.662 90)
       (effects (font (size 1.27 1.27)) hide)
@@
     (in_bom yes) (on_board yes)
     (property "Reference" "R204" (id 0) (at 147.32 97.79 90))
-    (property "Value" "1K" (id 1) (at 147.32 99.695 90))
+    (property "Value" "100" (id 1) (at 147.32 99.695 90))
     (property "Footprint" "Resistor_SMD:R_0603_1608Metric" (id 2) (at 147.32 96.393 90)
       (effects (font (size 1.27 1.27)) hide)
