File: hardware/s105/CAN.kicad_sch (KiCad schematic)
At the start: 7 parts, among them Q24 ., U7 SIT1042T/3

Commit message: #4 #5 #6 #8
Other:
- company: (none) -> rusEFI
- title: (none) -> s105
Changed lines of the file:
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@@
 (kicad_sch (version 20211123) (generator eeschema)
-  (paper "A4")
+  (paper "A3" portrait)
+  (title_block
+    (title "s105")
+    (rev "0.1")
+    (company "rusEFI")
+  )
   (junction (at 149.86 109.855) (diameter 0) (color 0 0 0 0)
   )
