File: hardware/s105/LM2902.kicad_sch (KiCad schematic)
At the start: 30 parts, among them U6 LM2902

Commit message: can, analog inputs
Changed lines of the file:
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@@
     (effects (font (size 1.27 1.27)) (justify left))
   )
-  (hierarchical_label "5V" (shape output) (at 68.58 52.705 90)
+  (hierarchical_label "5V" (shape input) (at 68.58 52.705 90)
     (effects (font (size 1.27 1.27)) (justify left))
   )

Commit message: закончила пока что
Parts:
- added D72: BAV99, Package_TO_SOT_SMD:SOT-23, symbol Diode:BAV99
Connections:
- net GND: now also D72.1 (K)
- net at C95.1, R274.2, R275.1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: now also U6.10 (+), U6.3 (+)
- net OUT2: now reaches R284.1, R285.2
- net OUT2: now also D72.3 (K)
- net at D57.3 (K), U6.8: no longer U6.3 (+)
- new net +5V: D72.2 (A)
Changed lines of the file:
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@@
   (junction (at 93.345 67.945) (diameter 0) (color 0 0 0 0)
   )
+  (junction (at 77.47 110.49) (diameter 0) (color 0 0 0 0)
+  )
   (junction (at 252.095 112.395) (diameter 0) (color 0 0 0 0)
   )
@@
   (junction (at 92.71 89.535) (diameter 0) (color 0 0 0 0)
   )
+  (junction (at 170.18 49.53) (diameter 0) (color 0 0 0 0)
+  )
   (junction (at 236.855 112.395) (diameter 0) (color 0 0 0 0)
   )
@@
   (junction (at 188.595 100.33) (diameter 0) (color 0 0 0 0)
   )
-  (junction (at 212.725 91.44) (diameter 0) (color 0 0 0 0)
+  (junction (at 111.125 67.945) (diameter 0) (color 0 0 0 0)
   )
   (junction (at 227.965 112.395) (diameter 0) (color 0 0 0 0)
@@
   (junction (at 133.985 89.535) (diameter 0) (color 0 0 0 0)
   )
+  (junction (at 77.47 89.535) (diameter 0) (color 0 0 0 0)
+  )
   (junction (at 133.985 70.485) (diameter 0) (color 0 0 0 0)
   )
@@
   (junction (at 204.47 114.935) (diameter 0) (color 0 0 0 0)
   )
-  (wire (pts (xy 212.725 91.44) (xy 212.725 67.945))
+  (wire (pts (xy 196.85 91.44) (xy 196.85 67.945))
+    (stroke (width 0) (type default) (color 0 0 0 0))
+  )
+  (wire (pts (xy 91.44 110.49) (xy 77.47 110.49))
     (stroke (width 0) (type default) (color 0 0 0 0))
   )
@@
     (stroke (width 0) (type default) (color 0 0 0 0))
   )
+  (wire (pts (xy 111.125 49.53) (xy 111.125 67.945))
+    (stroke (width 0) (type default) (color 0 0 0 0))
+  )
+  (wire (pts (xy 170.18 65.405) (xy 170.18 49.53))
+    (stroke (width 0) (type default) (color 0 0 0 0))
+  )
   (wire (pts (xy 172.085 102.87) (xy 172.72 102.87))
     (stroke (width 0) (type default) (color 0 0 0 0))
@@
     (stroke (width 0) (type default) (color 0 0 0 0))
   )
+  (wire (pts (xy 77.47 110.49) (xy 77.47 89.535))
+    (stroke (width 0) (type default) (color 0 0 0 0))
+  )
   (wire (pts (xy 125.095 89.535) (xy 113.03 89.535))
     (stroke (width 0) (type default) (color 0 0 0 0))
@@
     (stroke (width 0) (type default) (color 0 0 0 0))
   )
-  (wire (pts (xy 114.3 67.945) (xy 93.345 67.945))
+  (wire (pts (xy 114.3 67.945) (xy 111.125 67.945))
     (stroke (width 0) (type default) (color 0 0 0 0))
   )
@@
     (stroke (width 0) (type default) (color 0 0 0 0))
   )
-  (wire (pts (xy 162.56 91.44) (xy 212.725 91.44))
+  (wire (pts (xy 162.56 91.44) (xy 196.85 91.44))
     (stroke (width 0) (type default) (color 0 0 0 0))
   )
@@
     (stroke (width 0) (type default) (color 0 0 0 0))
   )
+  (wire (pts (xy 212.725 49.53) (xy 170.18 49.53))
+    (stroke (width 0) (type default) (color 0 0 0 0))
+  )
   (wire (pts (xy 154.305 70.485) (xy 154.305 74.295))
     (stroke (width 0) (type default) (color 0 0 0 0))
   )
+  (wire (pts (xy 111.125 67.945) (xy 93.345 67.945))
+    (stroke (width 0) (type default) (color 0 0 0 0))
+  )
   (wire (pts (xy 50.8 89.535) (xy 50.8 93.345))
     (stroke (width 0) (type default) (color 0 0 0 0))
   )
+  (wire (pts (xy 77.47 89.535) (xy 78.74 89.535))
+    (stroke (width 0) (type default) (color 0 0 0 0))
+  )
+  (wire (pts (xy 170.18 49.53) (xy 111.125 49.53))
+    (stroke (width 0) (type default) (color 0 0 0 0))
+  )
   (wire (pts (xy 85.09 67.945) (xy 93.345 67.945))
     (stroke (width 0) (type default) (color 0 0 0 0))
@@
     (stroke (width 0) (type default) (color 0 0 0 0))
   )
-  (wire (pts (xy 212.725 109.855) (xy 212.725 91.44))
-    (stroke (width 0) (type default) (color 0 0 0 0))
-  )
   (wire (pts (xy 166.37 102.87) (xy 172.085 102.87))
     (stroke (width 0) (type default) (color 0 0 0 0))
@@
     (stroke (width 0) (type default) (color 0 0 0 0))
   )
-  (wire (pts (xy 212.725 67.945) (xy 185.42 67.945))
+  (wire (pts (xy 196.85 67.945) (xy 185.42 67.945))
     (stroke (width 0) (type default) (color 0 0 0 0))
   )
@@
     (stroke (width 0) (type default) (color 0 0 0 0))
   )
-  (wire (pts (xy 74.93 89.535) (xy 78.74 89.535))
+  (wire (pts (xy 74.93 89.535) (xy 77.47 89.535))
     (stroke (width 0) (type default) (color 0 0 0 0))
   )
@@
     (stroke (width 0) (type default) (color 0 0 0 0))
   )
+  (wire (pts (xy 212.725 49.53) (xy 212.725 109.855))
+    (stroke (width 0) (type default) (color 0 0 0 0))
+  )
   (wire (pts (xy 113.03 73.025) (xy 113.03 78.105))
     (stroke (width 0) (type default) (color 0 0 0 0))
@@
   )
   (wire (pts (xy 137.16 70.485) (xy 133.985 70.485))
+    (stroke (width 0) (type default) (color 0 0 0 0))
+  )
+  (wire (pts (xy 74.295 110.49) (xy 77.47 110.49))
     (stroke (width 0) (type default) (color 0 0 0 0))
   )
@@
     (effects (font (size 1.27 1.27)) (justify left))
   )
+  (hierarchical_label "OUT2" (shape output) (at 91.44 110.49 0)
+    (effects (font (size 1.27 1.27)) (justify left))
+  )
   (hierarchical_label "IN" (shape output) (at 48.26 89.535 180)
     (effects (font (size 1.27 1.27)) (justify right))
@@
   )
   (hierarchical_label "5V" (shape input) (at 68.58 52.705 90)
+    (effects (font (size 1.27 1.27)) (justify left))
+  )
+  (hierarchical_label "GND" (shape output) (at 69.215 118.11 0)
     (effects (font (size 1.27 1.27)) (justify left))
   )
@@
     (pin "2")
   )
+  (symbol (lib_id "power:GND") (at 69.215 118.11 0) (unit 1)
+    (in_bom yes) (on_board yes) (fields_autoplaced)
+    (property "Reference" "#PWR0447" (id 0) (at 69.215 124.46 0)
+      (effects (font (size 1.27 1.27)) hide)
+    )
+    (property "Value" "GND" (id 1) (at 69.215 123.19 0))
+    (property "Footprint" "" (id 2) (at 69.215 118.11 0)
+      (effects (font (size 1.27 1.27)) hide)
+    )
+    (property "Datasheet" "" (id 3) (at 69.215 118.11 0)
+      (effects (font (size 1.27 1.27)) hide)
+    )
+    (pin "1")
+  )
   (symbol (lib_id "Amplifier_Operational:LM2902") (at 180.34 100.33 0) (unit 4)
     (in_bom yes) (on_board yes)
@@
     (pin "1")
   )
+  (symbol (lib_id "Diode:BAV99") (at 69.215 110.49 90) (unit 1)
+    (in_bom yes) (on_board yes) (fields_autoplaced)
+    (property "Reference" "D72" (id 0) (at 66.675 109.2199 90)
+      (effects (font (size 1.27 1.27)) (justify left))
+    )
+    (property "Value" "BAV99" (id 1) (at 66.675 111.7599 90)
+      (effects (font (size 1.27 1.27)) (justify left))
+    )
+    (property "Footprint" "Package_TO_SOT_SMD:SOT-23" (id 2) (at 81.915 110.49 0)
+      (effects (font (size 1.27 1.27)) hide)
+    )
+    (property "Datasheet" "https://assets.nexperia.com/documents/data-sheet/BAV99_SER.pdf" (id 3) (at 69.215 110.49 0)
+      (effects (font (size 1.27 1.27)) hide)
+    )
+    (pin "1")
+    (pin "2")
+    (pin "3")
+  )
   (symbol (lib_id "Device:R") (at 186.055 114.935 270) (mirror x) (unit 1)
     (in_bom yes) (on_board yes)
@@
     (pin "2")
   )
+  (symbol (lib_id "power:+5V") (at 69.215 102.87 0) (mirror y) (unit 1)
+    (in_bom yes) (on_board yes) (fields_autoplaced)
+    (property "Reference" "#PWR0446" (id 0) (at 69.215 106.68 0)
+      (effects (font (size 1.27 1.27)) hide)
+    )
+    (property "Value" "+5V" (id 1) (at 69.2151 99.06 90)
+      (effects (font (size 1.27 1.27)) (justify left))
+    )
+    (property "Footprint" "" (id 2) (at 69.215 102.87 0)
+      (effects (font (size 1.27 1.27)) hide)
+    )
+    (property "Datasheet" "" (id 3) (at 69.215 102.87 0)
+      (effects (font (size 1.27 1.27)) hide)
+    )
+    (pin "1")
+  )
   (symbol (lib_id "Device:C") (at 50.8 97.155 0) (unit 1)

Commit message: #4 #5 #6 #8
Other:
- company: (none) -> rusEFI
- title: (none) -> s105
Changed lines of the file:
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@@
 (kicad_sch (version 20211123) (generator eeschema)
-  (paper "A4")
+  (paper "A3" portrait)
+  (title_block
+    (title "s105")
+    (rev "0.1")
+    (company "rusEFI")
+  )
   (junction (at 212.725 114.935) (diameter 0) (color 0 0 0 0)
   )
