File: hardware/s105/OD_2A.kicad_sch (KiCad schematic)
At the start: 11 parts, among them Q11 BC847C

Commit message: #4 #5 #6 #8
Parts:
- renumbered C58 to C23, Q11 to Q2, R104 to R19, R105 to R20, R106 to R21, R107 to R22, R108 to R23, R109 to R24, R110 to R25, R111 to R26, VT12 to VT2
Other:
- company: (none) -> rusEFI
- title: (none) -> s105
Changed lines of the file:
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@@
 (kicad_sch (version 20211123) (generator eeschema)
-  (paper "A4")
+  (paper "A3" portrait)
+  (title_block
+    (title "s105")
+    (rev "0.1")
+    (company "rusEFI")
+  )
   (junction (at 180.34 81.28) (diameter 0) (color 0 0 0 0)
   )
@@
   (symbol (lib_id "Device:C") (at 189.23 69.85 0) (unit 1)
     (in_bom yes) (on_board yes)
-    (property "Reference" "C58" (id 0) (at 190.5 67.31 0)
+    (property "Reference" "C23" (id 0) (at 190.5 67.31 0)
       (effects (font (size 1.27 1.27)) (justify left))
     )
@@
   (symbol (lib_id "Device:R") (at 148.59 74.93 90) (unit 1)
     (in_bom yes) (on_board yes)
-    (property "Reference" "R105" (id 0) (at 148.59 72.39 90))
+    (property "Reference" "R20" (id 0) (at 148.59 72.39 90))
     (property "Value" "3K" (id 1) (at 148.59 77.47 90))
     (property "Footprint" "Resistor_SMD:R_0603_1608Metric" (id 2) (at 148.59 76.708 90)
@@
   (symbol (lib_id "Device:R") (at 167.64 86.36 0) (unit 1)
     (in_bom yes) (on_board yes) (fields_autoplaced)
-    (property "Reference" "R109" (id 0) (at 170.18 85.0899 0)
+    (property "Reference" "R24" (id 0) (at 170.18 85.0899 0)
       (effects (font (size 1.27 1.27)) (justify left))
     )
@@
   (symbol (lib_id "Device:R") (at 161.29 86.36 0) (unit 1)
     (in_bom yes) (on_board yes) (fields_autoplaced)
-    (property "Reference" "R108" (id 0) (at 163.83 85.0899 0)
+    (property "Reference" "R23" (id 0) (at 163.83 85.0899 0)
       (effects (font (size 1.27 1.27)) (justify left))
     )
@@
   (symbol (lib_id "power:GND") (at 189.23 73.66 0) (unit 1)
     (in_bom yes) (on_board yes) (fields_autoplaced)
-    (property "Reference" "#PWR0265" (id 0) (at 189.23 80.01 0)
+    (property "Reference" "#PWR0245" (id 0) (at 189.23 80.01 0)
       (effects (font (size 1.27 1.27)) hide)
     )
@@
   (symbol (lib_id "Device:R") (at 154.94 86.36 0) (unit 1)
     (in_bom yes) (on_board yes) (fields_autoplaced)
-    (property "Reference" "R107" (id 0) (at 157.48 85.0899 0)
+    (property "Reference" "R22" (id 0) (at 157.48 85.0899 0)
       (effects (font (size 1.27 1.27)) (justify left))
     )
@@
   (symbol (lib_id "Transistor_BJT:BC847") (at 138.43 81.28 0) (mirror y) (unit 1)
     (in_bom yes) (on_board yes) (fields_autoplaced)
-    (property "Reference" "Q11" (id 0) (at 133.35 80.0099 0)
+    (property "Reference" "Q2" (id 0) (at 133.35 80.0099 0)
       (effects (font (size 1.27 1.27)) (justify left))
     )
@@
   (symbol (lib_id "Device:R") (at 135.89 69.85 180) (unit 1)
     (in_bom yes) (on_board yes)
-    (property "Reference" "R104" (id 0) (at 133.35 69.85 90))
+    (property "Reference" "R19" (id 0) (at 133.35 69.85 90))
     (property "Value" "3K" (id 1) (at 138.43 69.85 90))
     (property "Footprint" "Resistor_SMD:R_0603_1608Metric" (id 2) (at 137.668 69.85 90)
@@
   (symbol (lib_id "Device:R") (at 180.34 86.36 180) (unit 1)
     (in_bom yes) (on_board yes)
-    (property "Reference" "R111" (id 0) (at 177.8 86.36 90))
+    (property "Reference" "R26" (id 0) (at 177.8 86.36 90))
     (property "Value" "51K" (id 1) (at 182.88 86.36 90))
     (property "Footprint" "Resistor_SMD:R_0603_1608Metric" (id 2) (at 182.118 86.36 90)
@@
   (symbol (lib_id "Device:R") (at 148.59 81.28 90) (unit 1)
     (in_bom yes) (on_board yes)
-    (property "Reference" "R106" (id 0) (at 148.59 78.74 90))
+    (property "Reference" "R21" (id 0) (at 148.59 78.74 90))
     (property "Value" "360R" (id 1) (at 148.59 83.82 90))
     (property "Footprint" "Resistor_SMD:R_0603_1608Metric" (id 2) (at 148.59 83.058 90)
@@
   (symbol (lib_id "Transistor_FET:IRFS4115") (at 158.75 74.93 0) (unit 1)
     (in_bom yes) (on_board yes) (fields_autoplaced)
-    (property "Reference" "VT12" (id 0) (at 165.1 73.6599 0)
+    (property "Reference" "VT2" (id 0) (at 165.1 73.6599 0)
       (effects (font (size 1.27 1.27)) (justify left))
     )
@@
   (symbol (lib_id "Device:R") (at 180.34 69.85 180) (unit 1)
     (in_bom yes) (on_board yes)
-    (property "Reference" "R110" (id 0) (at 177.8 69.85 90))
+    (property "Reference" "R25" (id 0) (at 177.8 69.85 90))
     (property "Value" "82K" (id 1) (at 182.88 69.85 90))
     (property "Footprint" "Resistor_SMD:R_0805_2012Metric" (id 2) (at 182.118 69.85 90)
