File: hardware/s105/OD_2A_2.kicad_sch (KiCad schematic)
At the start: 25 parts, among them Q17 BC847C

Commit message: +knock
Parts:
- R153: value 1k -> 100
- R211: value 10k -> 1k
Changed lines of the file:
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@@
     (in_bom yes) (on_board yes)
     (property "Reference" "R211" (id 0) (at 134.62 106.68 90))
-    (property "Value" "10k" (id 1) (at 132.08 106.68 90))
+    (property "Value" "1k" (id 1) (at 132.08 106.68 90))
     (property "Footprint" "Resistor_SMD:R_0603_1608Metric" (id 2) (at 130.302 106.68 90)
       (effects (font (size 1.27 1.27)) hide)
@@
     (in_bom yes) (on_board yes)
     (property "Reference" "R153" (id 0) (at 91.44 68.58 90))
-    (property "Value" "1k" (id 1) (at 93.98 68.58 90))
+    (property "Value" "100" (id 1) (at 93.98 68.58 90))
     (property "Footprint" "Resistor_SMD:R_0603_1608Metric" (id 2) (at 95.758 68.58 90)
       (effects (font (size 1.27 1.27)) hide)

Commit message: закончила пока что
Parts:
- added C49: C0603, Capacitor_SMD:C_0603_1608Metric, symbol Device:C
Connections:
- net GND: now also C49.2
- net OUT: now also C49.1
- no-connect marks 0 -> 1
Changed lines of the file:
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@@
   (junction (at 105.41 74.93) (diameter 0) (color 0 0 0 0)
   )
+  (junction (at 151.765 57.15) (diameter 0) (color 0 0 0 0)
+  )
   (junction (at 111.76 74.93) (diameter 0) (color 0 0 0 0)
   )
@@
   (junction (at 172.72 81.28) (diameter 0) (color 0 0 0 0)
   )
+  (no_connect (at 140.97 93.98))
   (wire (pts (xy 154.94 90.17) (xy 154.94 91.44))
     (stroke (width 0) (type default) (color 0 0 0 0))
@@
     (stroke (width 0) (type default) (color 0 0 0 0))
   )
+  (wire (pts (xy 151.765 57.15) (xy 143.51 57.15))
+    (stroke (width 0) (type default) (color 0 0 0 0))
+  )
   (wire (pts (xy 135.89 74.93) (xy 144.78 74.93))
     (stroke (width 0) (type default) (color 0 0 0 0))
@@
     (stroke (width 0) (type default) (color 0 0 0 0))
   )
-  (wire (pts (xy 147.32 57.15) (xy 143.51 57.15))
+  (wire (pts (xy 156.845 57.15) (xy 151.765 57.15))
     (stroke (width 0) (type default) (color 0 0 0 0))
   )
@@
     (effects (font (size 1.27 1.27)) (justify left))
   )
-  (hierarchical_label "OUT" (shape output) (at 147.32 57.15 0)
+  (hierarchical_label "OUT" (shape output) (at 156.845 57.15 0)
     (effects (font (size 1.27 1.27)) (justify left))
   )
@@
     )
     (property "Datasheet" "~" (id 3) (at 154.94 86.36 0)
+      (effects (font (size 1.27 1.27)) hide)
+    )
+    (pin "1")
+    (pin "2")
+  )
+  (symbol (lib_id "Device:C") (at 151.765 60.96 0) (unit 1)
+    (in_bom yes) (on_board yes)
+    (property "Reference" "C49" (id 0) (at 154.94 60.96 0)
+      (effects (font (size 1.27 1.27)) (justify left))
+    )
+    (property "Value" "C0603" (id 1) (at 153.67 63.5 0)
+      (effects (font (size 1.27 1.27)) (justify left))
+    )
+    (property "Footprint" "Capacitor_SMD:C_0603_1608Metric" (id 2) (at -137.033 143.51 90)
+      (effects (font (size 1.524 1.524)) hide)
+    )
+    (property "Datasheet" "" (id 3) (at 151.765 60.96 0)
+      (effects (font (size 1.524 1.524)) hide)
+    )
+    (property "PageName" "stm32f407_board" (id 4) (at 155.575 154.305 0)
+      (effects (font (size 1.524 1.524)) hide)
+    )
+    (property "Part #" "C0603" (id 5) (at -137.795 187.96 0)
+      (effects (font (size 1.27 1.27)) hide)
+    )
+    (property "VEND" "" (id 6) (at -137.795 187.96 0)
+      (effects (font (size 1.27 1.27)) hide)
+    )
+    (property "VEND#" "" (id 7) (at -137.795 187.96 0)
+      (effects (font (size 1.27 1.27)) hide)
+    )
+    (property "Manufacturer" "" (id 8) (at -137.795 187.96 0)
+      (effects (font (size 1.27 1.27)) hide)
+    )
+    (property "LCSC" "" (id 9) (at 151.765 60.96 0)
       (effects (font (size 1.27 1.27)) hide)
     )
@@
     (pin "3")
   )
+  (symbol (lib_id "power:GND") (at 151.765 64.77 0) (unit 1)
+    (in_bom yes) (on_board yes)
+    (property "Reference" "#PWR0350" (id 0) (at 151.765 71.12 0)
+      (effects (font (size 1.27 1.27)) hide)
+    )
+    (property "Value" "GND" (id 1) (at 149.86 69.215 0)
+      (effects (font (size 1.27 1.27)) (justify left))
+    )
+    (property "Footprint" "" (id 2) (at 151.765 64.77 0)
+      (effects (font (size 1.27 1.27)) hide)
+    )
+    (property "Datasheet" "" (id 3) (at 151.765 64.77 0)
+      (effects (font (size 1.27 1.27)) hide)
+    )
+    (pin "1")
+  )
   (symbol (lib_id "Transistor_FET:IRFS4115") (at 158.75 74.93 0) (unit 1)

Commit message: #4 #5 #6 #8
Connections:
- net at D15.3 (K), Q17.3 (C), R16.1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: now also D23.1 (K); no longer D23.2 (A)
- net at R157.1: now also D23.2 (A); no longer D23.1 (K)
Other:
- company: (none) -> rusEFI
- title: (none) -> s105
Changed lines of the file:
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@@
 (kicad_sch (version 20211123) (generator eeschema)
-  (paper "A4")
+  (paper "A3" portrait)
+  (title_block
+    (title "s105")
+    (rev "0.1")
+    (company "rusEFI")
+  )
   (junction (at 132.08 74.93) (diameter 0) (color 0 0 0 0)
   )
@@
     (pin "2")
   )
-  (symbol (lib_id "Diode:1N4148W") (at 124.46 74.93 0) (unit 1)
+  (symbol (lib_id "Diode:1N4148W") (at 124.46 74.93 0) (mirror y) (unit 1)
     (in_bom yes) (on_board yes)
     (property "Reference" "D23" (id 0) (at 124.46 68.58 0))
