File: hardware/s105/OD_2A_3.kicad_sch (KiCad schematic)
At the start: 7 parts

Commit message: закончила пока что
Connections:
- net OUT2: now reaches R163.1, VT18.3 (S)
Changed lines of the file:
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@@
   (junction (at 147.955 61.595) (diameter 0) (color 0 0 0 0)
+  )
+  (junction (at 128.905 78.105) (diameter 0) (color 0 0 0 0)
   )
   (junction (at 147.955 78.105) (diameter 0) (color 0 0 0 0)
@@
     (stroke (width 0) (type default) (color 0 0 0 0))
   )
-  (wire (pts (xy 128.905 76.835) (xy 128.905 79.375))
+  (wire (pts (xy 128.905 76.835) (xy 128.905 78.105))
+    (stroke (width 0) (type default) (color 0 0 0 0))
+  )
+  (wire (pts (xy 128.905 78.105) (xy 128.905 79.375))
     (stroke (width 0) (type default) (color 0 0 0 0))
   )
   (wire (pts (xy 156.845 61.595) (xy 156.845 62.865))
+    (stroke (width 0) (type default) (color 0 0 0 0))
+  )
+  (wire (pts (xy 98.425 78.105) (xy 128.905 78.105))
     (stroke (width 0) (type default) (color 0 0 0 0))
   )
@@
     (effects (font (size 1.27 1.27)) (justify left))
   )
+  (hierarchical_label "OUT2" (shape input) (at 98.425 78.105 180)
+    (effects (font (size 1.27 1.27)) (justify right))
+  )
   (symbol (lib_id "Transistor_FET:IRFS4115") (at 126.365 71.755 0) (unit 1)

Commit message: #4 #5 #6 #8
Other:
- company: (none) -> rusEFI
- title: (none) -> s105
Changed lines of the file:
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@@
 (kicad_sch (version 20211123) (generator eeschema)
-  (paper "A4")
+  (paper "A3" portrait)
+  (title_block
+    (title "s105")
+    (rev "0.1")
+    (company "rusEFI")
+  )
   (junction (at 103.505 71.755) (diameter 0) (color 0 0 0 0)
   )
