File: hardware/s105/VR.kicad_sch (KiCad schematic)
At the start: 17 parts, among them Q19 ., U3 case only

Commit message: закончила пока что
Parts:
- added D30: BAV99, Package_TO_SOT_SMD:SOT-23, symbol Diode:BAV99
Connections:
- net GND: now also D30.1 (K)
- net OUT: now also U3.1 (BOOT), D30.3 (K); no longer U3.5 (VCC)
- new net +3.3V: D30.2 (A)
- no-connect marks 0 -> 4
Changed lines of the file:
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@@
   (junction (at 189.865 107.315) (diameter 0) (color 0 0 0 0)
   )
+  (junction (at 121.285 95.885) (diameter 0) (color 0 0 0 0)
+  )
+  (no_connect (at 143.51 106.045))
+  (no_connect (at 102.87 90.805))
+  (no_connect (at 92.71 111.125))
+  (no_connect (at 92.71 100.965))
   (wire (pts (xy 153.67 106.045) (xy 153.67 120.65))
     (stroke (width 0) (type default) (color 0 0 0 0))
@@
     (stroke (width 0) (type default) (color 0 0 0 0))
   )
+  (wire (pts (xy 131.445 95.885) (xy 121.285 95.885))
+    (stroke (width 0) (type default) (color 0 0 0 0))
+  )
   (wire (pts (xy 171.45 107.315) (xy 165.1 107.315))
     (stroke (width 0) (type default) (color 0 0 0 0))
@@
     (stroke (width 0) (type default) (color 0 0 0 0))
   )
+  (wire (pts (xy 121.285 95.885) (xy 113.03 95.885))
+    (stroke (width 0) (type default) (color 0 0 0 0))
+  )
   (wire (pts (xy 189.865 107.315) (xy 198.12 107.315))
     (stroke (width 0) (type default) (color 0 0 0 0))
@@
     (stroke (width 0) (type default) (color 0 0 0 0))
   )
-  (wire (pts (xy 140.97 81.28) (xy 144.145 81.28))
+  (wire (pts (xy 123.19 78.105) (xy 121.285 78.105))
     (stroke (width 0) (type default) (color 0 0 0 0))
   )
@@
     (stroke (width 0) (type default) (color 0 0 0 0))
   )
-  (wire (pts (xy 113.03 111.125) (xy 115.57 111.125))
+  (wire (pts (xy 113.03 111.125) (xy 113.665 111.125))
     (stroke (width 0) (type default) (color 0 0 0 0))
   )
@@
     (stroke (width 0) (type default) (color 0 0 0 0))
   )
+  (wire (pts (xy 121.285 78.105) (xy 121.285 95.885))
+    (stroke (width 0) (type default) (color 0 0 0 0))
+  )
   (wire (pts (xy 123.19 103.505) (xy 113.03 103.505))
     (stroke (width 0) (type default) (color 0 0 0 0))
   )
   (wire (pts (xy 102.87 116.205) (xy 102.87 137.16))
-    (stroke (width 0) (type default) (color 0 0 0 0))
-  )
-  (wire (pts (xy 102.87 76.2) (xy 102.87 90.805))
-    (stroke (width 0) (type default) (color 0 0 0 0))
-  )
-  (wire (pts (xy 121.285 76.2) (xy 102.87 76.2))
     (stroke (width 0) (type default) (color 0 0 0 0))
   )
@@
     (effects (font (size 1.27 1.27)) (justify left))
   )
-  (hierarchical_label "GND" (shape output) (at 144.145 81.28 0)
+  (hierarchical_label "GND" (shape input) (at 113.665 111.125 0)
     (effects (font (size 1.27 1.27)) (justify left))
   )
@@
     (effects (font (size 1.27 1.27)) (justify left))
   )
-  (hierarchical_label "OUT" (shape output) (at 121.285 76.2 0)
+  (hierarchical_label "5V" (shape input) (at 165.1 67.945 90)
     (effects (font (size 1.27 1.27)) (justify left))
   )
-  (hierarchical_label "5V" (shape input) (at 165.1 67.945 90)
+  (hierarchical_label "OUT" (shape output) (at 131.445 95.885 0)
     (effects (font (size 1.27 1.27)) (justify left))
   )
@@
     (pin "2")
   )
+  (symbol (lib_id "power:+3.3V") (at 128.27 70.485 0) (mirror y) (unit 1)
+    (in_bom yes) (on_board yes) (fields_autoplaced)
+    (property "Reference" "#PWR0261" (id 0) (at 128.27 74.295 0)
+      (effects (font (size 1.27 1.27)) hide)
+    )
+    (property "Value" "+3.3V" (id 1) (at 128.27 65.405 0))
+    (property "Footprint" "" (id 2) (at 128.27 70.485 0)
+      (effects (font (size 1.27 1.27)) hide)
+    )
+    (property "Datasheet" "" (id 3) (at 128.27 70.485 0)
+      (effects (font (size 1.27 1.27)) hide)
+    )
+    (pin "1")
+  )
   (symbol (lib_id "Device:R") (at 165.1 128.8312 0) (mirror y) (unit 1)
     (in_bom yes) (on_board yes)
@@
     )
     (property "Datasheet" "" (id 3) (at 129.54 112.395 0)
+      (effects (font (size 1.27 1.27)) hide)
+    )
+    (pin "1")
+  )
+  (symbol (lib_id "power:GND") (at 128.27 85.725 0) (mirror y) (unit 1)
+    (in_bom yes) (on_board yes)
+    (property "Reference" "#PWR0258" (id 0) (at 128.27 92.075 0)
+      (effects (font (size 1.27 1.27)) hide)
+    )
+    (property "Value" "GND" (id 1) (at 128.27 89.535 0))
+    (property "Footprint" "" (id 2) (at 128.27 85.725 0)
+      (effects (font (size 1.27 1.27)) hide)
+    )
+    (property "Datasheet" "" (id 3) (at 128.27 85.725 0)
       (effects (font (size 1.27 1.27)) hide)
     )
@@
     (pin "2")
   )
+  (symbol (lib_id "Diode:BAV99") (at 128.27 78.105 270) (mirror x) (unit 1)
+    (in_bom yes) (on_board yes) (fields_autoplaced)
+    (property "Reference" "D30" (id 0) (at 130.81 76.8349 90)
+      (effects (font (size 1.27 1.27)) (justify left))
+    )
+    (property "Value" "BAV99" (id 1) (at 130.81 79.3749 90)
+      (effects (font (size 1.27 1.27)) (justify left))
+    )
+    (property "Footprint" "Package_TO_SOT_SMD:SOT-23" (id 2) (at 115.57 78.105 0)
+      (effects (font (size 1.27 1.27)) hide)
+    )
+    (property "Datasheet" "https://assets.nexperia.com/documents/data-sheet/BAV99_SER.pdf" (id 3) (at 128.27 78.105 0)
+      (effects (font (size 1.27 1.27)) hide)
+    )
+    (pin "1")
+    (pin "2")
+    (pin "3")
+  )
   (symbol (lib_id "Device:R") (at 165.1 88.265 0) (mirror y) (unit 1)
     (in_bom yes) (on_board yes)
@@
   (symbol (lib_id "Device:R") (at 123.19 108.585 0) (mirror x) (unit 1)
     (in_bom yes) (on_board yes)
-    (property "Reference" "R245" (id 0) (at 119.38 107.95 0))
-    (property "Value" "4.7k" (id 1) (at 118.745 109.855 0))
+    (property "Reference" "R245" (id 0) (at 119.38 107.315 0))
+    (property "Value" "4.7k" (id 1) (at 118.745 109.22 0))
     (property "Footprint" "Resistor_SMD:R_0603_1608Metric" (id 2) (at 121.412 108.585 90)
       (effects (font (size 1.27 1.27)) hide)
@@
     (pin "1")
   )
-  (symbol (lib_id "power:GND") (at 140.97 81.28 270) (mirror x) (unit 1)
-    (in_bom yes) (on_board yes)
-    (property "Reference" "#PWR014" (id 0) (at 134.62 81.28 0)
-      (effects (font (size 1.27 1.27)) hide)
-    )
-    (property "Value" "GND" (id 1) (at 137.2059 83.273 0)
-      (effects (font (size 1.27 1.27)) (justify left))
-    )
-    (property "Footprint" "" (id 2) (at 140.97 81.28 0)
-      (effects (font (size 1.27 1.27)) hide)
-    )
-    (property "Datasheet" "" (id 3) (at 140.97 81.28 0)
-      (effects (font (size 1.27 1.27)) hide)
-    )
-    (pin "1")
-  )
   (symbol (lib_id "Device:C") (at 165.1 114.3 0) (unit 1)
     (in_bom yes) (on_board yes)
@@
     (pin "2")
   )
-  (symbol (lib_id "power:GND") (at 115.57 111.125 0) (mirror y) (unit 1)
-    (in_bom yes) (on_board yes)
-    (property "Reference" "#PWR0385" (id 0) (at 115.57 117.475 0)
-      (effects (font (size 1.27 1.27)) hide)
-    )
-    (property "Value" "GND" (id 1) (at 117.563 114.8891 0)
-      (effects (font (size 1.27 1.27)) (justify left))
-    )
-    (property "Footprint" "" (id 2) (at 115.57 111.125 0)
-      (effects (font (size 1.27 1.27)) hide)
-    )
-    (property "Datasheet" "" (id 3) (at 115.57 111.125 0)
-      (effects (font (size 1.27 1.27)) hide)
-    )
-    (pin "1")
-  )
   (symbol (lib_id "Device:R") (at 189.865 113.665 0) (mirror x) (unit 1)

Commit message: #4 #5 #6 #8
Parts:
- removed Q19: ., Package_TO_SOT_SMD:SOT-23, symbol Transistor_BJT:BC847
- removed U3: case only, Package_SO:SOIC-8_3.9x4.9mm_P1.27mm, symbol Regulator_Controller:L6727
- added D73: ., Package_TO_SOT_SMD:SOT-23, symbol Diode:BAV99
- added U3: LM2903, Package_SO:SOIC-8_3.9x4.9mm_P1.27mm, symbol Comparator:LM2903
Connections:
- net 5V: now also U3.8 (V+)
- net GND: now also U3.4 (V-)
- net OUT: now also U3.1
- net at C46.1, R247.2, R248.2: now also D73.1 (K), U3.2 (-)
- net at C46.2, R246.1, R249.2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: now also D73.3 (K), U3.3 (+)
- net at R252.2, R253.1: now also R247.1, R251.2
Other:
- company: (none) -> rusEFI
- title: (none) -> s105
- moved on the sheet: C44, C45, C46, C47, C50, C51, D30, R245, R246, R247, R248, R249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
