File: hardware/s105/ak1sl2.kicad_sch (KiCad schematic)
At the start: 14 parts, among them U5 case only

Commit message: +knock
Parts:
- added R280: 300, Resistor_SMD:R_0603_1608Metric, symbol Device:R
- R264: value 3k -> 300
- R269: value 10k -> 1k
Connections:
- net GND: now also R280.2
- net at C94.1, R269.2, U5.6 (FB): now also R280.1
Changed lines of the file:
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@@
     (stroke (width 0) (type default) (color 0 0 0 0))
   )
-  (wire (pts (xy 97.79 93.98) (xy 99.695 93.98))
+  (wire (pts (xy 94.615 93.98) (xy 99.695 93.98))
     (stroke (width 0) (type default) (color 0 0 0 0))
   )
@@
   )
   (wire (pts (xy 169.926 115.57) (xy 173.736 115.57))
+    (stroke (width 0) (type default) (color 0 0 0 0))
+  )
+  (wire (pts (xy 125.73 123.19) (xy 132.08 123.19))
     (stroke (width 0) (type default) (color 0 0 0 0))
   )
@@
     (effects (font (size 1.27 1.27)) (justify right))
   )
-  (hierarchical_label "OUT" (shape output) (at 97.79 93.98 180)
+  (hierarchical_label "OUT" (shape output) (at 94.615 93.98 180)
     (effects (font (size 1.27 1.27)) (justify right))
   )
@@
     (pin "2")
   )
+  (symbol (lib_id "power:GND") (at 118.11 123.19 270) (mirror x) (unit 1)
+    (in_bom yes) (on_board yes)
+    (property "Reference" "#PWR0344" (id 0) (at 111.76 123.19 0)
+      (effects (font (size 1.27 1.27)) hide)
+    )
+    (property "Value" "GND" (id 1) (at 114.3459 125.183 0)
+      (effects (font (size 1.27 1.27)) (justify left))
+    )
+    (property "Footprint" "" (id 2) (at 118.11 123.19 0)
+      (effects (font (size 1.27 1.27)) hide)
+    )
+    (property "Datasheet" "" (id 3) (at 118.11 123.19 0)
+      (effects (font (size 1.27 1.27)) hide)
+    )
+    (pin "1")
+  )
   (symbol (lib_id "power:GND") (at 133.985 102.235 0) (mirror y) (unit 1)
     (in_bom yes) (on_board yes)
@@
     )
     (property "Datasheet" "~" (id 3) (at 181.61 117.475 0)
+      (effects (font (size 1.27 1.27)) hide)
+    )
+    (pin "1")
+    (pin "2")
+  )
+  (symbol (lib_id "Device:R") (at 121.92 123.19 270) (mirror x) (unit 1)
+    (in_bom yes) (on_board yes)
+    (property "Reference" "R280" (id 0) (at 121.92 120.65 90))
+    (property "Value" "300" (id 1) (at 121.92 125.73 90))
+    (property "Footprint" "Resistor_SMD:R_0603_1608Metric" (id 2) (at 121.92 124.968 90)
+      (effects (font (size 1.27 1.27)) hide)
+    )
+    (property "Datasheet" "~" (id 3) (at 121.92 123.19 0)
       (effects (font (size 1.27 1.27)) hide)
     )
@@
     (in_bom yes) (on_board yes)
     (property "Reference" "R264" (id 0) (at 146.685 91.44 90))
-    (property "Value" "3k" (id 1) (at 146.685 96.52 90))
+    (property "Value" "300" (id 1) (at 146.685 96.52 90))
     (property "Footprint" "Resistor_SMD:R_0603_1608Metric" (id 2) (at 146.685 95.758 90)
       (effects (font (size 1.27 1.27)) hide)
@@
   (symbol (lib_id "Device:R") (at 132.08 118.11 0) (mirror y) (unit 1)
     (in_bom yes) (on_board yes)
-    (property "Reference" "R269" (id 0) (at 134.62 117.475 0))
-    (property "Value" "10k" (id 1) (at 134.62 120.015 0))
+    (property "Reference" "R269" (id 0) (at 135.89 117.475 0))
+    (property "Value" "1k" (id 1) (at 135.89 119.38 0))
     (property "Footprint" "Resistor_SMD:R_0603_1608Metric" (id 2) (at 133.858 118.11 90)
       (effects (font (size 1.27 1.27)) hide)

Commit message: закончила пока что
Connections:
- net IN: now reaches R268.2
Other:
- note removed: "????????"
Changed lines of the file:
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@@
     (stroke (width 0) (type default) (color 0 0 0 0))
-  )
-  (text "????????\n" (at 200.025 128.27 180)
-    (effects (font (size 1.27 1.27)) (justify right bottom))
   )
   (hierarchical_label "3V3" (shape input) (at 171.45 95.25 90)
     (effects (font (size 1.27 1.27)) (justify left))
   )
+  (hierarchical_label "IN" (shape output) (at 201.93 127 0)
+    (effects (font (size 1.27 1.27)) (justify left))
+  )

Commit message: #4 #5 #6 #8
Other:
- company: (none) -> rusEFI
- title: (none) -> s105
Changed lines of the file:
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@@
 (kicad_sch (version 20211123) (generator eeschema)
-  (paper "A4")
+  (paper "A3" portrait)
+  (title_block
+    (title "s105")
+    (rev "0.1")
+    (company "rusEFI")
+  )
   (junction (at 99.695 93.98) (diameter 0) (color 0 0 0 0)
   )
