File: hardware/s105/analog.kicad_sch (KiCad schematic)
At the start: 82 parts

Commit message: заполняем плату дальше
Parts:
- added C64, C70: C0603, Capacitor_SMD:C_0603_1608Metric, symbol Device:C
- added C69, C72, C74, C75, C76, C77: 100nF, Capacitor_SMD:C_0603_1608Metric, symbol Device:C
Connections:
- net AC_Press: now also C76.2
- net AFR_1: now also C70.1
- net AFR_2: now also C64.1
- net CLT: now also C75.2
- net GND: now also C64.2, C69.1, C70.2, C72.1, C74.1, C75.1, C76.1, C77.1
- net IAT: now also C77.2
- net MAF: now also C72.2
- net MAP: now also C74.2
- net TPS: now also C69.2

Commit message: +knock
Parts:
- removed D46: 1N4148W, Diode_SMD:D_SOD-123, symbol Diode:1N4148W
- R215, R220: value 10k -> 1k
- R218, R222: value 60k -> 6k
- R233, R236: value 1k -> 100
- R72: value R0603 -> 1k
- R80: value 1K -> 100
Changed lines of the file:
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@@
     (effects (font (size 1.524 1.524) (thickness 0.3048) bold) (justify right))
   )
-  (hierarchical_label "PA2" (shape input) (at 191.77 177.165 180)
-    (effects (font (size 1.524 1.524) (thickness 0.3048) bold) (justify right))
-  )
   (hierarchical_label "PC4" (shape input) (at 128.27 107.315 0)
     (effects (font (size 1.524 1.524) (thickness 0.3048) bold) (justify left))
@@
   (symbol (lib_id "Device:R") (at 170.815 130.81 90) (mirror x) (unit 1)
     (in_bom yes) (on_board yes)
-    (property "Reference" "R72" (id 0) (at 170.815 132.842 90))
-    (property "Value" "R0603" (id 1) (at 170.815 130.81 90))
+    (property "Reference" "R72" (id 0) (at 170.815 128.27 90))
+    (property "Value" "1k" (id 1) (at 170.815 130.81 90))
     (property "Footprint" "Resistor_SMD:R_0603_1608Metric" (id 2) (at 112.395 189.992 90)
       (effects (font (size 1.524 1.524)) hide)
@@
     (in_bom yes) (on_board yes)
     (property "Reference" "R220" (id 0) (at 85.725 203.2 0))
-    (property "Value" "10k" (id 1) (at 84.455 205.105 0))
+    (property "Value" "1k" (id 1) (at 84.455 205.105 0))
     (property "Footprint" "Resistor_SMD:R_0603_1608Metric" (id 2) (at 90.043 203.2 90)
       (effects (font (size 1.27 1.27)) hide)
@@
     (in_bom yes) (on_board yes)
     (property "Reference" "R80" (id 0) (at 167.513 43.815 90))
-    (property "Value" "1K" (id 1) (at 169.545 43.815 90))
+    (property "Value" "100" (id 1) (at 169.545 43.815 90))
     (property "Footprint" "Resistor_SMD:R_0603_1608Metric" (id 2) (at 110.363 -14.605 90)
       (effects (font (size 1.524 1.524)) hide)
@@
     (in_bom yes) (on_board yes)
     (property "Reference" "R233" (id 0) (at 167.64 233.045 0))
-    (property "Value" "1k" (id 1) (at 166.37 234.95 0))
+    (property "Value" "100" (id 1) (at 166.37 234.95 0))
     (property "Footprint" "Resistor_SMD:R_0603_1608Metric" (id 2) (at 171.958 233.045 90)
       (effects (font (size 1.27 1.27)) hide)
@@
     (in_bom yes) (on_board yes)
     (property "Reference" "R218" (id 0) (at 103.505 63.5 0))
-    (property "Value" "60k" (id 1) (at 102.87 65.405 0))
+    (property "Value" "6k" (id 1) (at 102.87 65.405 0))
     (property "Footprint" "Resistor_SMD:R_0603_1608Metric" (id 2) (at 101.473 64.77 90)
       (effects (font (size 1.27 1.27)) hide)
@@
     (in_bom yes) (on_board yes)
     (property "Reference" "R222" (id 0) (at 105.41 202.565 0))
-    (property "Value" "60k" (id 1) (at 104.775 204.47 0))
+    (property "Value" "6k" (id 1) (at 104.775 204.47 0))
     (property "Footprint" "Resistor_SMD:R_0603_1608Metric" (id 2) (at 109.728 202.565 90)
       (effects (font (size 1.27 1.27)) hide)
@@
     (pin "1")
   )
-  (symbol (lib_id "Diode:1N4148W") (at 195.58 177.165 180) (unit 1)
-    (in_bom yes) (on_board yes) (fields_autoplaced)
-    (property "Reference" "D46" (id 0) (at 195.58 170.815 0))
-    (property "Value" "1N4148W" (id 1) (at 195.58 173.355 0))
-    (property "Footprint" "Diode_SMD:D_SOD-123" (id 2) (at 195.58 172.72 0)
-      (effects (font (size 1.27 1.27)) hide)
-    )
-    (property "Datasheet" "https://www.vishay.com/docs/85748/1n4148w.pdf" (id 3) (at 195.58 177.165 0)
-      (effects (font (size 1.27 1.27)) hide)
-    )
-    (pin "1")
-    (pin "2")
-  )
   (symbol (lib_id "Diode:BAV99") (at 130.175 196.85 270) (mirror x) (unit 1)
     (in_bom yes) (on_board yes) (fields_autoplaced)
@@
     (in_bom yes) (on_board yes)
     (property "Reference" "R215" (id 0) (at 83.82 62.865 0))
-    (property "Value" "10k" (id 1) (at 83.185 65.405 0))
+    (property "Value" "1k" (id 1) (at 83.185 65.405 0))
     (property "Footprint" "Resistor_SMD:R_0603_1608Metric" (id 2) (at 81.153 64.77 90)
       (effects (font (size 1.27 1.27)) hide)
@@
     (pin "2")
   )
-  (symbol (lib_id "power:+3.3V") (at 199.39 177.165 270) (mirror x) (unit 1)
-    (in_bom yes) (on_board yes) (fields_autoplaced)
-    (property "Reference" "#PWR0319" (id 0) (at 195.58 177.165 0)
-      (effects (font (size 1.27 1.27)) hide)
-    )
-    (property "Value" "+3.3V" (id 1) (at 203.2 177.1649 90)
-      (effects (font (size 1.27 1.27)) (justify left))
-    )
-    (property "Footprint" "" (id 2) (at 199.39 177.165 0)
-      (effects (font (size 1.27 1.27)) hide)
-    )
-    (property "Datasheet" "" (id 3) (at 199.39 177.165 0)
-      (effects (font (size 1.27 1.27)) hide)
-    )
-    (pin "1")
-  )
   (symbol (lib_id "power:GND") (at 153.035 69.85 0) (unit 1)
     (in_bom yes) (on_board yes)
@@
     (in_bom yes) (on_board yes)
     (property "Reference" "R236" (id 0) (at 175.895 233.045 0))
-    (property "Value" "1k" (id 1) (at 174.625 234.95 0))
+    (property "Value" "100" (id 1) (at 174.625 234.95 0))
     (property "Footprint" "Resistor_SMD:R_0603_1608Metric" (id 2) (at 180.213 233.045 90)
       (effects (font (size 1.27 1.27)) hide)

Commit message: can, analog inputs
Parts:
- added C100: C0603, Capacitor_SMD:C_0603_1608Metric, symbol Device:C
- added C101, C104, C48, C73, C78, C79, C88: 100nF, Capacitor_SMD:C_0603_1608Metric, symbol Device:C
- added C102, C103: NM, Capacitor_SMD:C_0603_1608Metric, symbol Device:C
- added D58, D59, D60, D61: BAV99, Package_TO_SOT_SMD:SOT-23, symbol Diode:BAV99
- added D62: NM, Diode_SMD:D_SOD-123, symbol Diode:1N4148W
- added R293, R299, R306: NM, Resistor_SMD:R_0603_1608Metric, symbol Device:R
- added R294, R310: 51k, Resistor_SMD:R_0603_1608Metric, symbol Device:R
- added R295: 4.7k, Resistor_SMD:R_0603_1608Metric, symbol Device:R
- added R296, R309: 33k, Resistor_SMD:R_0603_1608Metric, symbol Device:R
- added R297, R300, R301, R302, R307, R308, R312: NM, Resistor_SMD:R_1206_3216Metric, symbol Device:R
- added R298, R311: 4.7k, Resistor_SMD:R_1206_3216Metric, symbol Device:R
- added R303, R305: 300, Resistor_SMD:R_0603_1608Metric, symbol Device:R
Connections:
- net +3.3V: now also D58.2 (A), D59.2 (A), D60.2 (A), D61.2 (A)
- net GND: now also C100.2, C101.1, C102.1, C103.1, C104.1, C48.1, C73.1, C78.1, C79.1, C88.1, D58.1 (K), D59.1 (K), D60.1 (K), D61.1 (K), D62.1 (K), R296.1, R298.1, R301.1, R303.1, R305.1, R308.1, R309.1, R312.1
- new net: C100.1, D58.3 (K), R294.1, R295.2, R296.2
- new net 12V: R297.2, R300.2, R307.2, R311.2
- new net BOOT0: R293.1
- new net CAM_in: C88.2, R299.2, R300.1, R301.2
- new net DCNS: C73.2, R306.2, R307.1, R308.2
- new net NEW_PIN: C48.2, R302.2
- new net PB11: C103.2, D59.3 (K), R299.1, R303.2
- new net PB3: C101.2, D61.3 (K), R309.2, R310.1
- new net PC13: C102.2, D60.3 (K), R305.2, R306.1
- new net PD5: R295.1
- new net Prog_mode: C79.2, R293.2, R294.2, R297.1, R298.2
- new net Speed_in: C78.2, R310.2, R311.1, R312.2
- new net VBAT: C104.2, D62.2 (A), R302.1
Other:
- moved on the sheet: D47, D48, D53

Commit message: закончила пока что
Parts:
- removed D30, D50: BAV99, Package_TO_SOT_SMD:SOT-23, symbol Diode:BAV99
- added C113, C114, C115, C116, C117, C80, C81, C82, C83: 100nF, Capacitor_SMD:C_0603_1608Metric, symbol Device:C
- added D68, D69, D70, D71: BAV99, Package_TO_SOT_SMD:SOT-23, symbol Diode:BAV99
- added R318, R322, R324: 33k, Resistor_SMD:R_0603_1608Metric, symbol Device:R
- added R319, R325, R327: 51k, Resistor_SMD:R_0603_1608Metric, symbol Device:R
- added R320, R329, R332: 4.7k, Resistor_SMD:R_1206_3216Metric, symbol Device:R
- added R321, R328, R330, R331, R333: NM, Resistor_SMD:R_1206_3216Metric, symbol Device:R
- added R323: 300, Resistor_SMD:R_0603_1608Metric, symbol Device:R
- added R326: NM, Resistor_SMD:R_0603_1608Metric, symbol Device:R
Connections:
- net +3.3V: now also D68.2 (A), D69.2 (A), D70.2 (A), D71.2 (A)
- net 12V: now also R320.2, R328.2, R330.2, R332.2
- net GND: now also R209.2, C113.1, C114.1, C115.1, C116.1, C117.1, C80.1, C81.1, C82.1, C83.1, D68.1 (K), D69.1 (K), D70.1 (K), D71.1 (K), R318.1, R321.1, R322.1, R323.1, R324.1, R329.1, R331.1, R333.1
- net PA3: now also C36.2, D38.3 (K), R214.2; no longer C35.2, D37.3 (K), R164.2
- net PC0: now also C117.2
- net PC4: now also C35.2, D37.3 (K), R164.2; no longer C36.2, D38.3 (K), R214.2
- new net DIN1: C80.2, R319.2, R320.1, R321.2
- new net DIN5: C83.2, R327.2, R332.1, R333.2
- new net DPH2: C81.2, R326.2, R330.1, R331.2
- new net PC10: C116.2, D71.3 (K), R324.2, R327.1
- new net PC11: C115.2, D70.3 (K), R323.2, R326.1
- new net PC12: C113.2, D68.3 (K), R318.2, R319.1
- new net PD4: C114.2, D69.3 (K), R322.2, R325.1
- new net Start_req: C82.2, R325.2, R328.1, R329.2
Other:
- note added: "Это все к модулям OD"
- moved on the sheet: C100, C101, C102, C103, C104, C21, C34, C35, C36, C37, C38, C48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

Commit message: #4 #5 #6 #8
Connections:
- net 12V: now also R209.2
- net GND: no longer R209.2
Other:
- company: rusEFI.com -> rusEFI
- title: microRusEFI-2L -> s105
Changed lines of the file:
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@@
 (kicad_sch (version 20211123) (generator eeschema)
-  (paper "B")
+  (paper "A3" portrait)
   (title_block
-    (title "microRusEFI-2L")
+    (title "s105")
     (date "2022-04-10")
-    (rev "R0.6.0")
-    (company "rusEFI.com")
+    (rev "0.1")
+    (company "rusEFI")
     (comment 1 "Donald Becker")
     (comment 2 "AI6OD")
@@
   (hierarchical_label "PB11" (shape input) (at 332.74 207.01 180)
     (effects (font (size 1.524 1.524) (thickness 0.3048) bold) (justify right))
+  )
+  (hierarchical_label "12V" (shape input) (at 272.415 36.195 90)
+    (effects (font (size 1.27 1.27)) (justify left))
   )
   (hierarchical_label "PC4" (shape input) (at 101.6 61.595 0)
@@
     (pin "2")
   )
-  (symbol (lib_id "power:GND") (at 272.415 36.195 0) (mirror x) (unit 1)
-    (in_bom yes) (on_board yes)
-    (property "Reference" "#PWR0451" (id 0) (at 272.415 29.845 0)
-      (effects (font (size 1.27 1.27)) hide)
-    )
-    (property "Value" "GND" (id 1) (at 274.2241 31.8459 0)
-      (effects (font (size 1.27 1.27)) (justify right))
-    )
-    (property "Footprint" "" (id 2) (at 272.415 36.195 0)
-      (effects (font (size 1.27 1.27)) hide)
-    )
-    (property "Datasheet" "" (id 3) (at 272.415 36.195 0)
-      (effects (font (size 1.27 1.27)) hide)
-    )
-    (pin "1")
-  )
   (symbol (lib_id "power:+3.3V") (at 66.675 100.965 0) (unit 1)
