File: hardware/s105/s105.kicad_pcb (KiCad board)
At the start: 2 copper layers, 86 x 159 mm, 534 parts, among them J1 Conn_01x06, P1 368255-2, Q1 BC847C, Q10 BC847C, Q11 BC847C, Q12 BC847C, Q13 BC847C, Q14 BC847C, Q15 BC847C, Q16 BC847C, Q17 BC847C, Q18 BC847C, Q19 ., Q2 BC847C, Q20 BC847C, Q21 BC847C, Q22 BC847C, Q23 BC847C, Q24 ., Q3 BC847C, Q4 ., Q5 ., Q6 BC847C, Q7 BC847C, Q8 BC847C, Q9 BC847C, U1 case only, U2 STM32F427VGT6, U3 case only, U4 case only, U5 case only, U6 LM2902, U7 SIT1042T/3, X1 8MHz 20pF

Commit message: закончила пока что
Parts:
- added C105: NM, Capacitor_SMD:C_0603_1608Metric, F.Cu at (105.6, 134.8)
- added C106: C0603, Capacitor_SMD:C_0603_1608Metric, F.Cu at (125.5, 113.7)
- added C107: C1210, Capacitor_SMD:C_1210_3225Metric, F.Cu at (127.5, 105.5)
- added C108: C1210, Capacitor_SMD:C_1210_3225Metric, F.Cu at (127.5, 102.3)
- added C109: C0603, Capacitor_SMD:C_0603_1608Metric, F.Cu at (123.3, 104.8)
- added C110: C0805, Capacitor_SMD:C_0805_2012Metric, F.Cu at (106.1, 106.0)
- added C111: C0805, Capacitor_SMD:C_0805_2012Metric, F.Cu at (116.2, 104.8)
- added C112: C0603, Capacitor_SMD:C_0603_1608Metric, F.Cu at (114.4, 104.9)
- added C113: 100nF, Capacitor_SMD:C_0603_1608Metric, F.Cu at (94.1, 120.8)
- added C114: 100nF, Capacitor_SMD:C_0603_1608Metric, F.Cu at (106.6, 122.4)
- added C115: 100nF, Capacitor_SMD:C_0603_1608Metric, F.Cu at (101.6, 122.4)
- added C116: 100nF, Capacitor_SMD:C_0603_1608Metric, F.Cu at (111.3, 122.4)
- added C117: 100nF, Capacitor_SMD:C_0603_1608Metric, F.Cu at (105.0, 147.9)
- added C13: NM, Capacitor_SMD:C_0603_1608Metric, F.Cu at (102.1, 134.8)
- added D63: ., Diode_SMD:D_SOD-123, F.Cu at (119.8, 103.2)
- added D64: ., Diode_SMD:D_SOD-123, F.Cu at (131.4, 104.6)
- added D65: ., Diode_SMD:D_SMA, F.Cu at (107.7, 102.5)
- added D66: BAV99, Package_TO_SOT_SMD:SOT-23, F.Cu at (89.9, 124.1)
- added D67: BAV99, Package_TO_SOT_SMD:SOT-23, F.Cu at (94.4, 108.2)
- added D68: BAV99, Package_TO_SOT_SMD:SOT-23, F.Cu at (97.9, 117.5)
- added D69: BAV99, Package_TO_SOT_SMD:SOT-23, F.Cu at (107.7, 117.7)
- added D70: BAV99, Package_TO_SOT_SMD:SOT-23, F.Cu at (103.1, 117.7)
- added D71: BAV99, Package_TO_SOT_SMD:SOT-23, F.Cu at (112.2, 117.7)
- added D72: BAV99, Package_TO_SOT_SMD:SOT-23, F.Cu at (76.7, 159.3)
- added R304: NM, Resistor_SMD:R_0603_1608Metric, F.Cu at (105.1, 138.1)
- added R313: NM, Resistor_SMD:R_0603_1608Metric, F.Cu at (120.2, 115.9)
- added R314: NM, Resistor_SMD:R_0603_1608Metric, F.Cu at (120.2, 114.5)
- added R315: 4.7k, Resistor_SMD:R_0603_1608Metric, F.Cu at (106.4, 110.5)
- added R316: 4.7k, Resistor_SMD:R_0603_1608Metric, F.Cu at (116.1, 109.8)
- added R317: 1k, Resistor_SMD:R_0603_1608Metric, F.Cu at (114.5, 109.8)
- added R318: 33k, Resistor_SMD:R_0603_1608Metric, F.Cu at (94.1, 122.2)
- added R319: 51k, Resistor_SMD:R_0603_1608Metric, F.Cu at (96.6, 121.6)
- added R320: 4.7k, Resistor_SMD:R_1206_3216Metric, F.Cu at (97.1, 125.4)
- added R321: NM, Resistor_SMD:R_1206_3216Metric, F.Cu at (97.1, 127.5)
- added R322: 33k, Resistor_SMD:R_0603_1608Metric, F.Cu at (106.6, 120.9)
- added R323: 300, Resistor_SMD:R_0603_1608Metric, F.Cu at (101.6, 120.8)
- added R324: 33k, Resistor_SMD:R_0603_1608Metric, F.Cu at (111.3, 120.9)
- added R325: 51k, Resistor_SMD:R_0603_1608Metric, F.Cu at (108.8, 121.7)
- added R326: NM, Resistor_SMD:R_0603_1608Metric, F.Cu at (103.9, 121.6)
- added R327: 51k, Resistor_SMD:R_0603_1608Metric, F.Cu at (113.5, 121.7)
- added R328: NM, Resistor_SMD:R_1206_3216Metric, F.Cu at (107.4, 126.8)
- added R329: 4.7k, Resistor_SMD:R_1206_3216Metric, F.Cu at (107.4, 124.5)
- added R330: NM, Resistor_SMD:R_1206_3216Metric, F.Cu at (102.3, 126.8)
- added R331: NM, Resistor_SMD:R_1206_3216Metric, F.Cu at (102.3, 124.5)
- added R332: 4.7k, Resistor_SMD:R_1206_3216Metric, F.Cu at (112.3, 126.8)
- added R333: NM, Resistor_SMD:R_1206_3216Metric, F.Cu at (112.3, 124.5)
- added U8: case only, Package_SO:SOIC-8_3.9x4.9mm_P1.27mm, F.Cu at (122.3, 110.1)
- added U9: case only, Package_SO:SOIC-8_3.9x4.9mm_P1.27mm, F.Cu at (110.6, 108.1)
- added X2: NM, Crystal:Crystal_HC49-U_Vertical, F.Cu at (106.2, 131.4)
- C80, C81, C82, C83: value C0603 -> 100nF
- D11, D12, D13, D14, D16, D17, D18, D19, D20, D36, D4, D7: value BYG2OG -> .
- moved D21 4.25 mm to (115.2, 130.9)
- moved D56 4.25 mm to (111.8, 130.9)
- moved D24 3.62 mm to (108.5, 137.6)
- moved D5 3.47 mm to (110.7, 133.8)
- moved C98 3.18 mm to (77.5, 156.3)
- moved R285 2.94 mm to (75.3, 157.1)
- moved D1 2.60 mm to (95.5, 132.9)
- moved C92 2.27 mm to (79.3, 153.7)
- moved C1 1.94 mm to (93.9, 126.4)
- moved R9 1.94 mm to (93.9, 129.6)
- moved R12 1.70 mm to (92.1, 132.7)
- moved C93 1.16 mm to (93.0, 148.1)
- moved C2 1.14 mm to (92.6, 127.8)
- moved R13 1.14 mm to (91.0, 127.8)
- moved R292 1.12 mm to (82.2, 147.5)
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Connections:
- net /MCU/NRST renamed Net-(C5-Pad2)
- net /MCU/PA13 renamed /PA13
- net /MCU/PA14 renamed /PA14
- net /MCU/PB2-BOOT1 renamed /PB2
- net /MCU/PD8 renamed /PD8
- net Net-(R163-Pad1) renamed /OD 2A15/OUT2
- C35 pad 2: /PA3 -> /PC4
- C36 pad 2: /PC4 -> /PA3
- C80 pad 1: /DIN1 -> GND
- C80 pad 2: GND -> /DIN1
- C81 pad 1: /DPH2 -> GND
- C81 pad 2: GND -> /DPH2
- C82 pad 1: /Start_req -> GND
- C82 pad 2: GND -> /Start_req
- C83 pad 1: /DIN5 -> GND
- C83 pad 2: GND -> /DIN5
- C89 pad 1: /PA4 -> /PA5
- D14 pad 1: unconnected-(D14-Pad1) -> +12V
- D28 pad 1: /OD 2A14/OUT -> /IGN_swt
- D37 pad 3: /PA3 -> /PC4
- D38 pad 3: /PC4 -> /PA3
- Q15 pad 3: /PE11 -> /PE12
- R136 pad 1: /PE11 -> /PE12
- R137 pad 1: /PE11 -> /PE12
- R142 pad 1: /PE12 -> /PE13
- R143 pad 2: /PE12 -> /PE13
- R164 pad 2: /PA3 -> /PC4
- R209 pad 2: unconnected-(R209-Pad2) -> GND
- R214 pad 2: /PC4 -> /PA3
- R244 pad 2: /OD 2A22/3V3 -> +3.3V
- R261 pad 1: /PA4 -> /PA5
- R262 pad 2: /PA4 -> /PA5
- R263 pad 1: /PA4 -> /PA5
- R264 pad 2: /PA4 -> /PA5
- R268 pad 2: unconnected-(R268-Pad2) -> /OD 2A24/IN
- R284 pad 1: Net-(R284-Pad1) -> /PE4
- R285 pad 2: Net-(R284-Pad1) -> /PE4
- R57 pad 1: Net-(R57-Pad1) -> /OD 2A24/IN
- R7 pad 1: /PA15 -> /PC8
- R8 pad 2: /PA15 -> /PC8
- U2 pad 2: /MCU/PE3 -> /PE3
- U2 pad 20: /MCU/VSSA -> GND
- U2 pad 3: /MCU/PE4 -> /PE4
- U2 pad 30: /MCU/PA5 -> /PA5
- U2 pad 35: /MCU/PB0 -> /PB0
- U2 pad 36: /MCU/PB1 -> /PB1
- U2 pad 43: /MCU/PE12 -> /PE12
- U2 pad 44: /MCU/PE13 -> /PE13
- U2 pad 53: /MCU/PB14 -> /PB14
- U2 pad 54: /MCU/PB15 -> /PB15
- U2 pad 77: /MCU/PA15 -> /PA15
- U2 pad 78: /MCU/PC10 -> /PC10
- U2 pad 79: /MCU/PC11 -> /PC11
- U2 pad 8: unconnected-(U2-Pad8) -> Net-(U2-Pad8)
- U2 pad 80: /MCU/PC12 -> /PC12
- U2 pad 81: /MCU/PD0 -> /PD0
- U2 pad 85: /MCU/PD4 -> /PD4
- U2 pad 9: unconnected-(U2-Pad9) -> Net-(U2-Pad9)
- U3 pad 1: unconnected-(U3-Pad1) -> /PB10
- U3 pad 5: /PB10 -> unconnected-(U3-Pad5)
- U6 pad 10: unconnected-(U6-Pad10) -> Net-(C95-Pad1)
- U6 pad 3: Net-(D57-Pad3) -> Net-(C95-Pad1)
- U7 pad 5: /CAN A1/3V3 -> +3.3V
- VT6 pad 3: Net-(R57-Pad1) -> /OD 2A24/IN

Commit message: #4 #5 #6 #8
Parts:
- removed Q19: ., Package_TO_SOT_SMD:SOT-23
- added D73: ., Package_TO_SOT_SMD:SOT-23, F.Cu at (76.1, 176.8)
- U3: value case only -> LM2903
Connections:
- R247 pad 1: Net-(R247-Pad1) -> Net-(R252-Pad2)
- R251 pad 2: Net-(R247-Pad1) -> Net-(R252-Pad2)
