File: hardware/s105/soic-8_NM.kicad_sch (KiCad schematic)
At the start: 15 parts, among them Q18 BC847C, Q8 BC847C, U1 case only

Commit message: закончила пока что
Parts:
- added D50: BAV99, Package_TO_SOT_SMD:SOT-23, symbol Diode:BAV99
Connections:
- net GND: now also D50.1 (K)
- net OUT: now also D50.3 (K)
- new net +3.3V: D50.2 (A)
Changed lines of the file:
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@@
   (junction (at 175.26 87.63) (diameter 0) (color 0 0 0 0)
   )
+  (junction (at 216.535 87.63) (diameter 0) (color 0 0 0 0)
+  )
   (junction (at 189.865 111.125) (diameter 0) (color 0 0 0 0)
   )
@@
     (stroke (width 0) (type default) (color 0 0 0 0))
   )
+  (wire (pts (xy 216.535 87.63) (xy 216.535 80.645))
+    (stroke (width 0) (type default) (color 0 0 0 0))
+  )
   (wire (pts (xy 201.93 116.205) (xy 201.93 118.11))
     (stroke (width 0) (type default) (color 0 0 0 0))
@@
     (stroke (width 0) (type default) (color 0 0 0 0))
   )
+  (wire (pts (xy 216.535 80.645) (xy 222.25 80.645))
+    (stroke (width 0) (type default) (color 0 0 0 0))
+  )
   (wire (pts (xy 201.93 99.06) (xy 201.93 106.045))
     (stroke (width 0) (type default) (color 0 0 0 0))
   )
   (wire (pts (xy 189.23 92.71) (xy 189.23 99.06))
+    (stroke (width 0) (type default) (color 0 0 0 0))
+  )
+  (wire (pts (xy 216.535 87.63) (xy 227.33 87.63))
     (stroke (width 0) (type default) (color 0 0 0 0))
   )
@@
     (effects (font (size 1.27 1.27)) (justify left))
   )
-  (hierarchical_label "OUT" (shape output) (at 216.535 87.63 0)
+  (hierarchical_label "OUT" (shape output) (at 222.25 80.645 0)
     (effects (font (size 1.27 1.27)) (justify left))
   )
@@
     )
     (property "Datasheet" "" (id 3) (at 151.13 125.73 0)
+      (effects (font (size 1.27 1.27)) hide)
+    )
+    (pin "1")
+  )
+  (symbol (lib_id "power:+3.3V") (at 232.41 80.01 0) (mirror y) (unit 1)
+    (in_bom yes) (on_board yes) (fields_autoplaced)
+    (property "Reference" "#PWR0330" (id 0) (at 232.41 83.82 0)
+      (effects (font (size 1.27 1.27)) hide)
+    )
+    (property "Value" "+3.3V" (id 1) (at 232.41 74.93 0))
+    (property "Footprint" "" (id 2) (at 232.41 80.01 0)
+      (effects (font (size 1.27 1.27)) hide)
+    )
+    (property "Datasheet" "" (id 3) (at 232.41 80.01 0)
       (effects (font (size 1.27 1.27)) hide)
     )
@@
     (pin "1")
     (pin "2")
+  )
+  (symbol (lib_id "Diode:BAV99") (at 232.41 87.63 270) (mirror x) (unit 1)
+    (in_bom yes) (on_board yes) (fields_autoplaced)
+    (property "Reference" "D50" (id 0) (at 234.95 86.3599 90)
+      (effects (font (size 1.27 1.27)) (justify left))
+    )
+    (property "Value" "BAV99" (id 1) (at 234.95 88.8999 90)
+      (effects (font (size 1.27 1.27)) (justify left))
+    )
+    (property "Footprint" "Package_TO_SOT_SMD:SOT-23" (id 2) (at 219.71 87.63 0)
+      (effects (font (size 1.27 1.27)) hide)
+    )
+    (property "Datasheet" "https://assets.nexperia.com/documents/data-sheet/BAV99_SER.pdf" (id 3) (at 232.41 87.63 0)
+      (effects (font (size 1.27 1.27)) hide)
+    )
+    (pin "1")
+    (pin "2")
+    (pin "3")
   )
   (symbol (lib_id "Device:C") (at 111.76 114.3 0) (unit 1)
@@
     (pin "2")
   )
+  (symbol (lib_id "power:GND") (at 232.41 95.25 0) (mirror y) (unit 1)
+    (in_bom yes) (on_board yes) (fields_autoplaced)
+    (property "Reference" "#PWR0329" (id 0) (at 232.41 101.6 0)
+      (effects (font (size 1.27 1.27)) hide)
+    )
+    (property "Value" "GND" (id 1) (at 232.41 100.33 0))
+    (property "Footprint" "" (id 2) (at 232.41 95.25 0)
+      (effects (font (size 1.27 1.27)) hide)
+    )
+    (property "Datasheet" "" (id 3) (at 232.41 95.25 0)
+      (effects (font (size 1.27 1.27)) hide)
+    )
+    (pin "1")
+  )
   (symbol (lib_id "power:GND") (at 143.51 82.55 270) (mirror x) (unit 1)

Commit message: #4 #5 #6 #8
Other:
- company: (none) -> rusEFI
- title: (none) -> s105
Changed lines of the file:
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@@
 (kicad_sch (version 20211123) (generator eeschema)
-  (paper "A4")
+  (paper "A3" portrait)
+  (title_block
+    (title "s105")
+    (rev "0.1")
+    (company "rusEFI")
+  )
   (junction (at 111.76 110.49) (diameter 0) (color 0 0 0 0)
   )
