File: hardware/s105/stm32.kicad_sch (KiCad schematic)
At the start: 22 parts, among them J1 Conn_01x06, U2 STM32F427VGT6, X1 8MHz 20pF

Commit message: can, analog inputs
Parts:
- removed C13: 10nF, Capacitor_SMD:C_0603_1608Metric, symbol Device:C
- R15: value 10K -> 51K
Connections:
- net VBAT: now reaches U2.6 (VBAT)
Changed lines of the file:
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@@
   (junction (at 113.03 97.79) (diameter 0) (color 0 0 0 0)
   )
-  (junction (at 158.75 63.5) (diameter 0) (color 0 0 0 0)
-  )
   (junction (at 170.18 229.87) (diameter 0) (color 0 0 0 0)
   )
@@
   (junction (at 108.585 97.79) (diameter 0) (color 0 0 0 0)
   )
+  (junction (at 115.57 102.87) (diameter 0) (color 0 0 0 0)
+  )
   (wire (pts (xy 170.18 229.87) (xy 170.815 229.87))
     (stroke (width 0) (type default) (color 0 0 0 0))
@@
     (stroke (width 0) (type default) (color 0 0 0 0))
   )
-  (wire (pts (xy 152.4 63.5) (xy 158.75 63.5))
+  (wire (pts (xy 107.95 102.87) (xy 115.57 102.87))
+    (stroke (width 0) (type default) (color 0 0 0 0))
+  )
+  (wire (pts (xy 152.4 63.5) (xy 167.64 63.5))
     (stroke (width 0) (type default) (color 0 0 0 0))
   )
@@
   )
   (wire (pts (xy 270.51 111.76) (xy 262.89 111.76))
-    (stroke (width 0) (type default) (color 0 0 0 0))
-  )
-  (wire (pts (xy 158.75 63.5) (xy 167.64 63.5))
     (stroke (width 0) (type default) (color 0 0 0 0))
   )
@@
     (effects (font (size 1.524 1.524) (thickness 0.3048) bold) (justify left))
   )
+  (hierarchical_label "BOOT0" (shape input) (at 107.95 102.87 180)
+    (effects (font (size 1.524 1.524) (thickness 0.3048) bold) (justify right))
+  )
   (hierarchical_label "PC7" (shape input) (at 186.69 201.93 0)
     (effects (font (size 1.524 1.524) (thickness 0.3048) bold) (justify left))
@@
   (hierarchical_label "PE10" (shape input) (at 140.97 166.37 180)
     (effects (font (size 1.524 1.524) (thickness 0.3048) bold) (justify right))
+  )
+  (hierarchical_label "VBAT" (shape input) (at 156.21 88.9 90)
+    (effects (font (size 1.524 1.524) (thickness 0.3048) bold) (justify left))
   )
   (hierarchical_label "PA13" (shape input) (at 186.69 130.81 0)
@@
     (pin "1")
     (pin "2")
-  )
-  (symbol (lib_id "Device:C") (at 158.75 59.69 0) (unit 1)
-    (in_bom yes) (on_board yes)
-    (property "Reference" "C13" (id 0) (at 160.02 57.15 0)
-      (effects (font (size 1.27 1.27)) (justify left))
-    )
-    (property "Value" "10nF" (id 1) (at 159.385 62.23 0)
-      (effects (font (size 1.27 1.27)) (justify left))
-    )
-    (property "Footprint" "Capacitor_SMD:C_0603_1608Metric" (id 2) (at 133.477 -7.62 90)
-      (effects (font (size 1.524 1.524)) hide)
-    )
-    (property "Datasheet" "" (id 3) (at 222.885 -8.255 0)
-      (effects (font (size 1.524 1.524)) hide)
-    )
-    (property "Part #" "C0603C103K1RACTU" (id 4) (at 0 119.38 0)
-      (effects (font (size 1.27 1.27)) hide)
-    )
-    (property "VEND" "DIGI" (id 5) (at 0 119.38 0)
-      (effects (font (size 1.27 1.27)) hide)
-    )
-    (property "VEND#" "399-3189-1-ND" (id 6) (at 0 119.38 0)
-      (effects (font (size 1.27 1.27)) hide)
-    )
-    (property "Manufacturer" "KEMET" (id 7) (at 0 119.38 0)
-      (effects (font (size 1.27 1.27)) hide)
-    )
-    (property "LCSC" "C57112" (id 8) (at 158.75 59.69 0)
-      (effects (font (size 1.27 1.27)) hide)
-    )
-    (pin "1")
-    (pin "2")
-  )
-  (symbol (lib_id "power:GND") (at 158.75 55.88 180) (unit 1)
-    (in_bom yes) (on_board yes)
-    (property "Reference" "#PWR0136" (id 0) (at 158.75 55.88 0)
-      (effects (font (size 0.762 0.762)) hide)
-    )
-    (property "Value" "GND" (id 1) (at 158.75 54.102 0)
-      (effects (font (size 0.762 0.762)) hide)
-    )
-    (property "Footprint" "" (id 2) (at 158.75 55.88 0)
-      (effects (font (size 1.524 1.524)))
-    )
-    (property "Datasheet" "" (id 3) (at 158.75 55.88 0)
-      (effects (font (size 1.524 1.524)))
-    )
-    (pin "1")
   )
   (symbol (lib_id "Device:C") (at 166.37 80.01 0) (unit 1)
@@
     (in_bom yes) (on_board yes)
     (property "Reference" "R15" (id 0) (at 119.38 111.252 90))
-    (property "Value" "10K" (id 1) (at 119.38 109.22 90))
+    (property "Value" "51K" (id 1) (at 119.38 109.22 90))
     (property "Footprint" "Resistor_SMD:R_0603_1608Metric" (id 2) (at 60.96 168.402 90)
       (effects (font (size 1.524 1.524)) hide)
@@
       (effects (font (size 1.27 1.27)) hide)
     )
-    (pin "1")
-  )
-  (symbol (lib_id "power:PWR_FLAG") (at 156.21 88.9 0) (unit 1)
-    (in_bom yes) (on_board yes)
-    (property "Reference" "#FLG0101" (id 0) (at 156.21 86.995 0)
-      (effects (font (size 1.27 1.27)) hide)
-    )
-    (property "Value" "PWR_FLAG" (id 1) (at 156.21 84.5058 0)
-      (effects (font (size 1.27 1.27)) hide)
-    )
-    (property "Footprint" "" (id 2) (at 156.21 88.9 0)
-      (effects (font (size 1.27 1.27)) hide)
-    )
-    (property "Datasheet" "~" (id 3) (at 156.21 88.9 0)
-      (effects (font (size 1.27 1.27)) hide)
-    )

Commit message: закончила пока что
Parts:
- added C105, C13: NM, Capacitor_SMD:C_0603_1608Metric, symbol Device:C
- added R304: NM, Resistor_SMD:R_0603_1608Metric, symbol Device:R
- added X2: NM, Crystal:Crystal_HC49-U_Vertical, symbol Device:Crystal
Connections:
- net GND: now also C105.2, C13.2
- net at U2.8 (PC14): now also C105.1, X2.2
- net at U2.9 (PC15): now also R304.1
- net NRST: no longer names the net of C5.2, R14.2, U2.14 (NRST)
- new net: C13.1, R304.2, X2.1
- no-connect marks 0 -> 1

Commit message: #4 #5 #6 #8
Other:
- company: rusEFI.com -> rusEFI
- title: microRusEFI-2L -> s105
Changed lines of the file:
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@@
 (kicad_sch (version 20211123) (generator eeschema)
-  (paper "B")
+  (paper "A3" portrait)
   (title_block
-    (title "microRusEFI-2L")
+    (title "s105")
     (date "2022-04-10")
-    (rev "R0.6.0")
-    (company "rusEFI.com")
+    (rev "0.1")
+    (company "rusEFI")
     (comment 1 "Donald Becker")
     (comment 2 "AI6OD")
